File: eagle/BYOG_Shield.sch (EAGLE design)
At the start: 1 part, among them U1 ARDUINOR3-NOIOREF-NOTEXT

Commit message: COMPLETE & EXPRESS versions of PCB files added
Added in EXPRESS and COMPLETE version of the EAGLE files to
complete/refer to.
Use EXPRESS to jumpstart the routing task. Good luck and have fun!
Parts:
- added IC1, IC2: 74HC595N, AISCube_BYOG:74HC595N
- added LED1: (no value), AISCube_BYOG:LED/0805
- added R1, R2, R3: (no value), AISCube_BYOG:RESISTOR0805-RES
- added U$1, U$2: PB_SMTFITTING, AISCube_BYOG:PB_SMTFITTING
- added U$3: 8X8DM_2088AS, AISCube_BYOG:8X8DM_2088AS
Connections:
- new net 5V: IC1P.VCC, IC2P.VCC, R2.2, R3.2, U1.5V
- new net GND: IC1P.GND, IC2P.GND, LED1.C, U1.GND1, U1.GND2
- new net N$1: R1.1, U1.D10
- new net N$10: IC1A.QD, U$3.R4
- new net N$11: IC1A.QE, U$3.R5
- new net N$12: IC1A.QF, U$3.R6
- new net N$13: IC1A.QG, U$3.R7
- new net N$14: IC1A.QH, U$3.R8
- new net N$15: IC1A.QA, U$3.R1
- new net N$16: IC2A.QB, U$3.C2
- new net N$17: IC2A.QC, U$3.C3
- new net N$18: IC2A.QD, U$3.C4
- new net N$19: IC2A.QE, U$3.C5
- new net N$20: IC2A.QF, U$3.C6
- new net N$21: IC2A.QG, U$3.C7
- new net N$22: IC2A.QH, U$3.C8
- new net N$23: IC2A.QA, U$3.C1
- new net N$5: LED1.A, R1.2
- new net N$6: R2.1, U$1.1
- new net N$7: R3.1, U$2.1
- new net N$8: IC1A.QB, U$3.R2
- new net N$9: IC1A.QC, U$3.R3
- new net PB1: U1.D5
- new net PB2: U1.D6
